Commit message: feat: el chasis se apoya en sus orugas en vez de atravesar el suelo
Las orugas del URDF son su banda entre las dos poleas y el chasis cuelga
de tres juntas virtuales (altura, cabeceo, balanceo) que publica
chasis_node desde las elevaciones y la geometria del propio URDF.

File: ros2_ws/src/starcrawler_description/urdf/starcrawler.urdf.xacro (robot description, xacro)
@@ -9,7 +9,13 @@
     a los grados de encoder del firmware (180 deg = horizontal; las orugas
     FL y RR van espejadas, 360-a, como documenta el TFG).
+  Cada oruga es la banda alrededor de dos poleas: la activa en el pivote (la
+  que mueve el RMD, su radio es el wheel_radius de la odometria) y la pasiva
+  en la punta. El chasis cuelga de tres juntas virtuales (altura, cabeceo y
+  balanceo) que publica chasis_node: al bajar una oruga el chasis se levanta
+  sobre ella en vez de atravesar el suelo. Con todo a cero, orugas en llano.
   DIMENSIONES: valores iniciales APROXIMADOS. Medir en el robot y ajustar aqui
-  (todo son propiedades xacro, se cambia en un sitio).
-  Referencia: cajas envolventes de los STEP de ControlHORUFinalBoss/CAD (mm):
+  (todo son propiedades xacro, se cambia en un sitio; chasis_node las lee del
+  propio URDF). Referencia: cajas envolventes de los STEP de
+  ControlHORUFinalBoss/CAD (mm):
       Chasis.STEP ................. 1300 x 80 x 400
       Correa v2 (oruga) ........... 622 x 327 x 80
@@ -29,10 +35,22 @@
   <xacro:property name="base_height"  value="0.10"/>   <!-- Z             -->
   <xacro:property name="base_mass"    value="20.0"/>   <!-- kg, aprox      -->
-  <xacro:property name="arm_length"   value="0.36"/>   <!-- pivote a punta -->
+  <!-- Poleas de la oruga: activa del CAD (0.15279/2, = wheel_radius) y
+       pasiva de diametro 83 -->
+  <xacro:property name="pulley_radius" value="0.0764"/>
+  <xacro:property name="tip_radius"    value="0.0415"/>
+  <xacro:property name="arm_length"   value="0.36"/>   <!-- entre ejes de poleas -->
   <xacro:property name="arm_width"    value="0.08"/>
-  <xacro:property name="arm_height"   value="0.09"/>
   <xacro:property name="arm_mass"     value="3.0"/>
-  <!-- Altura del pivote sobre el suelo (con las orugas horizontales) -->
-  <xacro:property name="pivot_height" value="0.09"/>
+  <xacro:property name="belt_thickness" value="0.012"/>
+  <!-- Tramos de banda: tangentes a las dos poleas, inclinados belt_angle -->
+  <xacro:property name="belt_angle"  value="${asin((pulley_radius - tip_radius) / arm_length)}"/>
+  <xacro:property name="belt_length" value="${arm_length * cos(belt_angle)}"/>
+  <xacro:property name="belt_x"
+      value="${arm_length/2 + (pulley_radius + tip_radius - belt_thickness)/2 * sin(belt_angle)}"/>
+  <xacro:property name="belt_z"
+      value="${(pulley_radius + tip_radius - belt_thickness)/2 * cos(belt_angle)}"/>
+  <!-- Altura del pivote sobre el suelo con las orugas en llano: la banda
+       apoya bajo la polea activa -->
+  <xacro:property name="pivot_height" value="${pulley_radius}"/>
   <!-- Limite de recorrido: encoder 90..270 deg -> +-90 deg de elevacion -->
   <xacro:property name="arm_limit"    value="${pi/2}"/>
@@ -61,8 +79,26 @@
   <!-- base_footprint: proyeccion en el suelo, raiz para Nav2 -->
   <link name="base_footprint"/>
-  <joint name="base_joint" type="fixed">
+  <!-- Juntas virtuales del apoyo: las publica chasis_node. La altura se
+       mide desde la de las orugas en llano, para que cero sea reposo. -->
+  <joint name="chassis_lift_joint" type="prismatic">
     <parent link="base_footprint"/>
+    <child link="chassis_lift_link"/>
+    <origin xyz="0 0 ${pivot_height}"/>
+    <axis xyz="0 0 1"/>
+    <limit lower="0.0" upper="${arm_length + tip_radius}" effort="0" velocity="1"/>
+  </joint>
+  <link name="chassis_lift_link"/>
+  <joint name="chassis_pitch_joint" type="revolute">
+    <parent link="chassis_lift_link"/>
+    <child link="chassis_pitch_link"/>
+    <axis xyz="0 1 0"/>
+    <limit lower="${-pi/2}" upper="${pi/2}" effort="0" velocity="1"/>
+  </joint>
+  <link name="chassis_pitch_link"/>
+  <joint name="chassis_roll_joint" type="revolute">
+    <parent link="chassis_pitch_link"/>
     <child link="base_link"/>
-    <origin xyz="0 0 ${pivot_height}"/>
+    <axis xyz="1 0 0"/>
+    <limit lower="${-pi/2}" upper="${pi/2}" effort="0" velocity="1"/>
   </joint>
   <link name="base_link">
@@ -81,4 +117,6 @@
        El eje de giro se elige para que POSITIVO = brazo levantado en las
        cuatro orugas: delanteras giran sobre -Y, traseras sobre +Y.
+       El pivote es el eje de la polea activa; chasis_node reconoce las
+       poleas como los dos cilindros del link.
   -->
   <xacro:macro name="crawler" params="name x_sign y_sign material">
@@ -94,12 +132,27 @@
     <link name="${name}_link">
       <visual>
-        <!-- el brazo sale del pivote hacia fuera del chasis -->
-        <origin xyz="${x_sign*arm_length/2} 0 0"/>
-        <geometry><box size="${arm_length} ${arm_width} ${arm_height}"/></geometry>
+        <origin rpy="${pi/2} 0 0"/>
+        <geometry><cylinder radius="${pulley_radius}" length="${arm_width}"/></geometry>
+        <material name="${material}"/>
+      </visual>
+      <visual>
+        <origin xyz="${x_sign*arm_length} 0 0" rpy="${pi/2} 0 0"/>
+        <geometry><cylinder radius="${tip_radius}" length="${arm_width}"/></geometry>
+        <material name="${material}"/>
+      </visual>
+      <!-- tramo de arriba y tramo de abajo de la banda -->
+      <visual>
+        <origin xyz="${x_sign*belt_x} 0 ${belt_z}" rpy="0 ${x_sign*belt_angle} 0"/>
+        <geometry><box size="${belt_length} ${arm_width} ${belt_thickness}"/></geometry>
+        <material name="${material}"/>
+      </visual>
+      <visual>
+        <origin xyz="${x_sign*belt_x} 0 ${-belt_z}" rpy="0 ${-x_sign*belt_angle} 0"/>
+        <geometry><box size="${belt_length} ${arm_width} ${belt_thickness}"/></geometry>
         <material name="${material}"/>
       </visual>
       <collision>
         <origin xyz="${x_sign*arm_length/2} 0 0"/>
-        <geometry><box size="${arm_length} ${arm_width} ${arm_height}"/></geometry>
+        <geometry><box size="${arm_length} ${arm_width} ${2*pulley_radius}"/></geometry>
       </collision>
       <inertial>
@@ -107,6 +160,6 @@
         <mass value="${arm_mass}"/>
         <inertia
-          ixx="${arm_mass*(arm_width*arm_width+arm_height*arm_height)/12.0}" ixy="0.0" ixz="0.0"
-          iyy="${arm_mass*(arm_length*arm_length+arm_height*arm_height)/12.0}" iyz="0.0"
+          ixx="${arm_mass*(arm_width*arm_width+4*pulley_radius*pulley_radius)/12.0}" ixy="0.0" ixz="0.0"
+          iyy="${arm_mass*(arm_length*arm_length+4*pulley_radius*pulley_radius)/12.0}" iyz="0.0"
           izz="${arm_mass*(arm_length*arm_length+arm_width*arm_width)/12.0}"/>
       </inertial>

Commit message: sim: mundo_node, marcadores y arg mundo:= en el launch
Con un mundo cargado mundo_node publica la pose verdadera, las juntas del
chasis y /mundo/estado; RViz pinta la arena. Probado en vivo en escalon.

File: ros2_ws/src/starcrawler_description/urdf/starcrawler.urdf.xacro (robot description, xacro)
@@ -79,5 +79,6 @@
   <!-- base_footprint: proyeccion en el suelo, raiz para Nav2 -->
   <link name="base_footprint"/>
-  <!-- Juntas virtuales del apoyo: las publica chasis_node. La altura se
+  <!-- Juntas virtuales del apoyo: las publica chasis_node, o mundo_node con
+       un mundo cargado (entonces la altura es la del terreno). La altura se
        mide desde la de las orugas en llano, para que cero sea reposo. -->
   <joint name="chassis_lift_joint" type="prismatic">
@@ -86,5 +87,5 @@
     <origin xyz="0 0 ${pivot_height}"/>
     <axis xyz="0 0 1"/>
-    <limit lower="0.0" upper="${arm_length + tip_radius}" effort="0" velocity="1"/>
+    <limit lower="-0.6" upper="2.0" effort="0" velocity="1"/>
   </joint>
   <link name="chassis_lift_link"/>

Commit message: description: el aspecto de Horu (caja roja, chapas amarillas, banda negra)
Chapas, tacos, tapacubos, faros y soportes van en links fijos: los parsers
de chasis_node y del contacto solo leen los cilindros del brazo. El visor de
MuJoCo usa los mismos colores.

File: ros2_ws/src/starcrawler_description/urdf/starcrawler.urdf.xacro (robot description, xacro)
@@ -43,4 +43,11 @@
   <xacro:property name="arm_mass"     value="3.0"/>
   <xacro:property name="belt_thickness" value="0.012"/>
+  <!-- Aspecto (solo visual): tacos de la banda y chapas laterales -->
+  <xacro:property name="lug_count"  value="12"/>
+  <xacro:property name="lug_length" value="0.012"/>
+  <xacro:property name="lug_height" value="0.010"/>
+  <xacro:property name="plate_t"    value="0.006"/>
+  <xacro:property name="plate_r1"   value="${pulley_radius*0.82}"/>
+  <xacro:property name="plate_r2"   value="${tip_radius*0.9}"/>
   <!-- Tramos de banda: tangentes a las dos poleas, inclinados belt_angle -->
   <xacro:property name="belt_angle"  value="${asin((pulley_radius - tip_radius) / arm_length)}"/>
@@ -60,5 +67,13 @@
   <xacro:property name="arm_effort"   value="60.0"/>
   <!-- ─── Materiales ──────────────────────────────────────────────────── -->
-  <material name="sc_chasis"><color rgba="0.20 0.20 0.20 1.0"/></material>
+  <!-- Los de Horu (fotos): caja roja, chapas amarillas y banda de goma
+       negra. Cada brazo conserva su color en el tapacubos. -->
+  <material name="sc_chasis"><color rgba="0.80 0.05 0.05 1.0"/></material>
+  <material name="sc_tapa">  <color rgba="0.68 0.03 0.03 1.0"/></material>
+  <material name="sc_chapa"> <color rgba="1.00 0.82 0.00 1.0"/></material>
+  <material name="sc_goma">  <color rgba="0.07 0.07 0.07 1.0"/></material>
+  <material name="sc_metal"> <color rgba="0.75 0.76 0.78 1.0"/></material>
+  <material name="sc_negro"> <color rgba="0.12 0.12 0.12 1.0"/></material>
+  <material name="sc_luz">   <color rgba="0.95 0.95 0.85 1.0"/></material>
   <material name="sc_fr">    <color rgba="0.22 0.53 0.90 1.0"/></material>
   <material name="sc_fl">    <color rgba="0.00 0.51 0.00 1.0"/></material>
@@ -135,10 +150,10 @@
         <origin rpy="${pi/2} 0 0"/>
         <geometry><cylinder radius="${pulley_radius}" length="${arm_width}"/></geometry>
-        <material name="${material}"/>
+        <material name="sc_goma"/>
       </visual>
       <visual>
         <origin xyz="${x_sign*arm_length} 0 0" rpy="${pi/2} 0 0"/>
         <geometry><cylinder radius="${tip_radius}" length="${arm_width}"/></geometry>
-        <material name="${material}"/>
+        <material name="sc_goma"/>
       </visual>
       <!-- tramo de arriba y tramo de abajo de la banda -->
@@ -146,10 +161,10 @@
         <origin xyz="${x_sign*belt_x} 0 ${belt_z}" rpy="0 ${x_sign*belt_angle} 0"/>
         <geometry><box size="${belt_length} ${arm_width} ${belt_thickness}"/></geometry>
-        <material name="${material}"/>
+        <material name="sc_goma"/>
       </visual>
       <visual>
         <origin xyz="${x_sign*belt_x} 0 ${-belt_z}" rpy="0 ${-x_sign*belt_angle} 0"/>
         <geometry><box size="${belt_length} ${arm_width} ${belt_thickness}"/></geometry>
-        <material name="${material}"/>
+        <material name="sc_goma"/>
       </visual>
       <collision>
@@ -167,8 +182,125 @@
     </link>
   </xacro:macro>
+  <!-- Tacos de la banda, n por tramo (recursivo). side = +1 arriba, -1 abajo -->
+  <xacro:macro name="tacos" params="n x_sign side">
+    <xacro:if value="${n > 0}">
+      <xacro:property name="ang" value="${side*x_sign*belt_angle}"/>
+      <xacro:property name="u" value="${(n - 0.5)/lug_count*belt_length - belt_length/2}"/>
+      <xacro:property name="off" value="${belt_thickness/2 + lug_height/2}"/>
+      <visual>
+        <origin xyz="${x_sign*belt_x + u*cos(ang) + side*off*sin(ang)} 0 ${side*belt_z - u*sin(ang) + side*off*cos(ang)}"
+                rpy="0 ${ang} 0"/>
+        <geometry><box size="${lug_length} ${arm_width} ${lug_height}"/></geometry>
+        <material name="sc_goma"/>
+      </visual>
+      <xacro:tacos n="${n-1}" x_sign="${x_sign}" side="${side}"/>
+    </xacro:if>
+  </xacro:macro>
+  <xacro:macro name="chapa" params="x_sign lado">
+    <visual>
+      <origin xyz="${x_sign*arm_length/2} ${lado*(arm_width/2 + plate_t/2)} 0"/>
+      <geometry><box size="${arm_length} ${plate_t} ${2*plate_r2}"/></geometry>
+      <material name="sc_chapa"/>
+    </visual>
+    <visual>
+      <origin xyz="0 ${lado*(arm_width/2 + plate_t/2)} 0" rpy="${pi/2} 0 0"/>
+      <geometry><cylinder radius="${plate_r1}" length="${plate_t}"/></geometry>
+      <material name="sc_chapa"/>
+    </visual>
+    <visual>
+      <origin xyz="${x_sign*arm_length} ${lado*(arm_width/2 + plate_t/2)} 0" rpy="${pi/2} 0 0"/>
+      <geometry><cylinder radius="${plate_r2}" length="${plate_t}"/></geometry>
+      <material name="sc_chapa"/>
+    </visual>
+  </xacro:macro>
+  <!-- Chapas amarillas, tacos, tensor y tapacubos de cada oruga, en un link
+       fijo: chasis_node y el contacto solo leen los cilindros del brazo -->
+  <xacro:macro name="crawler_deco" params="name x_sign y_sign material">
+    <joint name="${name}_deco_joint" type="fixed">
+      <parent link="${name}_link"/>
+      <child link="${name}_deco"/>
+    </joint>
+    <link name="${name}_deco">
+      <xacro:tacos n="${lug_count}" x_sign="${x_sign}" side="1"/>
+      <xacro:tacos n="${lug_count}" x_sign="${x_sign}" side="-1"/>
+      <xacro:chapa x_sign="${x_sign}" lado="1"/>
+      <xacro:chapa x_sign="${x_sign}" lado="-1"/>
+      <visual>
+        <origin xyz="${x_sign*arm_length} ${y_sign*(arm_width/2 + plate_t + 0.006)} 0" rpy="${pi/2} 0 0"/>
+        <geometry><cylinder radius="0.012" length="0.012"/></geometry>
+        <material name="sc_metal"/>
+      </visual>
+      <visual>
+        <origin xyz="${x_sign*(arm_length - 0.085)} ${y_sign*(arm_width/2 + plate_t + 0.006)} 0.012"/>
+        <geometry><box size="0.07 0.012 0.022"/></geometry>
+        <material name="sc_metal"/>
+      </visual>
+      <visual>
+        <origin xyz="0 ${y_sign*(arm_width/2 + plate_t + 0.008)} 0" rpy="${pi/2} 0 0"/>
+        <geometry><cylinder radius="0.03" length="0.016"/></geometry>
+        <material name="sc_metal"/>
+      </visual>
+      <visual>
+        <origin xyz="0 ${y_sign*(arm_width/2 + plate_t + 0.017)} 0" rpy="${pi/2} 0 0"/>
+        <geometry><cylinder radius="0.014" length="0.003"/></geometry>
+        <material name="${material}"/>
+      </visual>
+    </link>
+  </xacro:macro>
   <xacro:crawler name="crawler_fr" x_sign="1"  y_sign="-1" material="sc_fr"/>
   <xacro:crawler name="crawler_fl" x_sign="1"  y_sign="1"  material="sc_fl"/>
   <xacro:crawler name="crawler_rr" x_sign="-1" y_sign="-1" material="sc_rr"/>
   <xacro:crawler name="crawler_rl" x_sign="-1" y_sign="1"  material="sc_rl"/>
+  <xacro:crawler_deco name="crawler_fr" x_sign="1"  y_sign="-1" material="sc_fr"/>
+  <xacro:crawler_deco name="crawler_fl" x_sign="1"  y_sign="1"  material="sc_fl"/>
+  <xacro:crawler_deco name="crawler_rr" x_sign="-1" y_sign="-1" material="sc_rr"/>
+  <xacro:crawler_deco name="crawler_rl" x_sign="-1" y_sign="1"  material="sc_rl"/>
+  <!-- Detalles de la caja: tapa, faros, asas y soportes de los brazos -->
+  <xacro:macro name="faro" params="y">
+    <visual>
+      <origin xyz="${base_length/2 + 0.01} ${y} -0.01" rpy="0 ${pi/2} 0"/>
+      <geometry><cylinder radius="0.022" length="0.02"/></geometry>
+      <material name="sc_negro"/>
+    </visual>
+    <visual>
+      <origin xyz="${base_length/2 + 0.021} ${y} -0.01" rpy="0 ${pi/2} 0"/>
+      <geometry><cylinder radius="0.016" length="0.003"/></geometry>
+      <material name="sc_luz"/>
+    </visual>
+  </xacro:macro>
+  <xacro:macro name="soporte" params="xs ys">
+    <visual>
+      <origin xyz="${xs*(base_length/2 - 0.06)} ${ys*(base_width/2 - 0.05)} ${-base_height/2 - 0.012}"/>
+      <geometry><box size="0.10 0.07 0.024"/></geometry>
+      <material name="sc_metal"/>
+    </visual>
+  </xacro:macro>
+  <joint name="chasis_deco_joint" type="fixed">
+    <parent link="base_link"/>
+    <child link="chasis_deco"/>
+  </joint>
+  <link name="chasis_deco">
+    <visual>
+      <origin xyz="0 0 ${base_height/2 + 0.002}"/>
+      <geometry><box size="${base_length - 0.02} ${base_width - 0.02} 0.004"/></geometry>
+      <material name="sc_tapa"/>
+    </visual>
+    <xacro:faro y="0.09"/>
+    <xacro:faro y="-0.09"/>
+    <visual>
+      <origin xyz="0.12 ${base_width/2 + 0.006} 0.015"/>
+      <geometry><box size="0.06 0.012 0.03"/></geometry>
+      <material name="sc_negro"/>
+    </visual>
+    <visual>
+      <origin xyz="0.12 ${-base_width/2 - 0.006} 0.015"/>
+      <geometry><box size="0.06 0.012 0.03"/></geometry>
+      <material name="sc_negro"/>
+    </visual>
+    <xacro:soporte xs="1"  ys="1"/>
+    <xacro:soporte xs="1"  ys="-1"/>
+    <xacro:soporte xs="-1" ys="1"/>
+    <xacro:soporte xs="-1" ys="-1"/>
+  </link>
   <!-- ─── Sitio para la IMU ───────────────────────────────────────────────
        En el TFG la MPU9250 iba en el frontal del chasis. Con PC a bordo lo

Commit message: orugas: los tacos se mueven con la banda (bandas_node)
Cada tramo y cada arco de polea es una junta cuyo limite es el paso de
taco; bandas_node la mueve con la velocidad de banda de /starcrawler/state,
asi que vale con el simulador, el ESP32 o el driver serie.

File: ros2_ws/src/starcrawler_description/urdf/starcrawler.urdf.xacro (robot description, xacro)
@@ -182,18 +182,67 @@
     </link>
   </xacro:macro>
-  <!-- Tacos de la banda, n por tramo (recursivo). side = +1 arriba, -1 abajo -->
-  <xacro:macro name="tacos" params="n x_sign side">
+  <!-- Tacos que se mueven. Como van equiespaciados, basta desplazarlos lo
+       que avanza la banda modulo un paso de taco: cada tramo es una junta
+       prismatica (0..paso) y cada arco alrededor de una polea, una de giro
+       (0..paso angular). Las publica bandas_node; el limite superior de
+       cada junta es su periodo. -->
+  <xacro:property name="lug_pitch" value="${belt_length/lug_count}"/>
+  <!-- n tacos a lo largo de un tramo, en el marco del tramo -->
+  <xacro:macro name="tacos_tramo" params="n side">
     <xacro:if value="${n > 0}">
-      <xacro:property name="ang" value="${side*x_sign*belt_angle}"/>
-      <xacro:property name="u" value="${(n - 0.5)/lug_count*belt_length - belt_length/2}"/>
-      <xacro:property name="off" value="${belt_thickness/2 + lug_height/2}"/>
-      <visual>
-        <origin xyz="${x_sign*belt_x + u*cos(ang) + side*off*sin(ang)} 0 ${side*belt_z - u*sin(ang) + side*off*cos(ang)}"
-                rpy="0 ${ang} 0"/>
+      <visual>
+        <origin xyz="${(n - 0.5)*lug_pitch - belt_length/2} 0 ${side*(belt_thickness/2 + lug_height/2)}"/>
         <geometry><box size="${lug_length} ${arm_width} ${lug_height}"/></geometry>
         <material name="sc_goma"/>
       </visual>
-      <xacro:tacos n="${n-1}" x_sign="${x_sign}" side="${side}"/>
+      <xacro:tacos_tramo n="${n-1}" side="${side}"/>
     </xacro:if>
+  </xacro:macro>
+  <!-- Tacos del arco de una polea (los de la mitad por donde abraza la
+       banda). extremo = -1 polea activa, +1 polea de la punta -->
+  <xacro:macro name="tacos_arco" params="k n r x_sign extremo">
+    <xacro:if value="${n - k > 0}">
+      <xacro:property name="th" value="${2*pi*k/n}"/>
+      <xacro:if value="${extremo*(x_sign*cos(th) - sin(belt_angle)) >= 0}">
+        <visual>
+          <origin xyz="${(r + lug_height/2)*cos(th)} 0 ${(r + lug_height/2)*sin(th)}"
+                  rpy="0 ${pi/2 - th} 0"/>
+          <geometry><box size="${lug_length} ${arm_width} ${lug_height}"/></geometry>
+          <material name="sc_goma"/>
+        </visual>
+      </xacro:if>
+      <xacro:tacos_arco k="${k+1}" n="${n}" r="${r}" x_sign="${x_sign}" extremo="${extremo}"/>
+    </xacro:if>
+  </xacro:macro>
+  <xacro:macro name="banda_movil" params="name x_sign">
+    <xacro:macro name="tramo" params="lado side">
+      <joint name="${name}_tacos_${lado}_joint" type="prismatic">
+        <parent link="${name}_link"/>
+        <child link="${name}_tacos_${lado}"/>
+        <origin xyz="${x_sign*belt_x} 0 ${side*belt_z}" rpy="0 ${side*x_sign*belt_angle} 0"/>
+        <axis xyz="${side} 0 0"/>
+        <limit lower="0" upper="${lug_pitch}" effort="0" velocity="1"/>
+      </joint>
+      <link name="${name}_tacos_${lado}">
+        <xacro:tacos_tramo n="${lug_count}" side="${side}"/>
+      </link>
+    </xacro:macro>
+    <xacro:tramo lado="arriba" side="1"/>
+    <xacro:tramo lado="abajo" side="-1"/>
+    <xacro:macro name="arco" params="lado x r extremo">
+      <xacro:property name="n" value="${int(2*pi*r/lug_pitch + 0.5)}"/>
+      <joint name="${name}_tacos_${lado}_joint" type="revolute">
+        <parent link="${name}_link"/>
+        <child link="${name}_tacos_${lado}"/>
+        <origin xyz="${x} 0 0"/>
+        <axis xyz="0 1 0"/>
+        <limit lower="0" upper="${2*pi/n}" effort="0" velocity="10"/>
+      </joint>
+      <link name="${name}_tacos_${lado}">
+        <xacro:tacos_arco k="0" n="${n}" r="${r}" x_sign="${x_sign}" extremo="${extremo}"/>
+      </link>
+    </xacro:macro>
+    <xacro:arco lado="polea" x="0" r="${pulley_radius}" extremo="-1"/>
+    <xacro:arco lado="punta" x="${x_sign*arm_length}" r="${tip_radius}" extremo="1"/>
   </xacro:macro>
   <xacro:macro name="chapa" params="x_sign lado">
@@ -214,5 +263,5 @@
     </visual>
   </xacro:macro>
-  <!-- Chapas amarillas, tacos, tensor y tapacubos de cada oruga, en un link
+  <!-- Chapas amarillas, tensor y tapacubos de cada oruga, en un link
        fijo: chasis_node y el contacto solo leen los cilindros del brazo -->
   <xacro:macro name="crawler_deco" params="name x_sign y_sign material">
@@ -221,7 +270,6 @@
       <child link="${name}_deco"/>
     </joint>
+    <xacro:banda_movil name="${name}" x_sign="${x_sign}"/>
     <link name="${name}_deco">
-      <xacro:tacos n="${lug_count}" x_sign="${x_sign}" side="1"/>
-      <xacro:tacos n="${lug_count}" x_sign="${x_sign}" side="-1"/>
       <xacro:chapa x_sign="${x_sign}" lado="1"/>
       <xacro:chapa x_sign="${x_sign}" lado="-1"/>
